File: kicad_atlas_joint.kicad_sch (KiCad schematic)
At the start: 7 parts, among them IC1 AS5600, J1 Conn_01x07_Pin, J2 Conn_01x06_Pin, U1 STM32F411CEUx, U2 INA226, U3 LM2596S-3.3

Commit message: changes
Parts:
- removed J1: Conn_01x07_Pin, symbol Connector:Conn_01x07_Pin
- removed J2: Conn_01x06_Pin, symbol Connector:Conn_01x06_Pin
- added C1, C3: 10uF, symbol Device:C_Polarized_Small
- added C2, C4, C6, C7, C8: 100nF, symbol Device:C_Small
- added C5: 10uF, symbol Device:C_Small
- added J1: Screw_Terminal_01x07, symbol Connector:Screw_Terminal_01x07
- added J3: Screw_Terminal_01x06, symbol Connector:Screw_Terminal_01x06
- added R1, R2, R7, R8: 10kOhm, symbol Device:R_Small
- added R3: 1kOhm, symbol Device:R_Small
- added R4: 1.7kOhm, symbol Device:R_Small
- added R5, R6: 4.7kOhm, symbol Device:R_Small
- added SW1: SW_Push, symbol Switch:SW_Push
Connections:
- net CONN2_GND, CONN1_GND, LM2596_GND is gone; now on net GND: U3.3 (GND)
- net LM2596_GND is gone; now on net GND: A1.1 (GND), IC1.4 (GND), IC1.5 (PGO), U1.23 (VSS), U1.35 (VSS), U1.47 (VSS), U1.49 (VSS), U2.1 (A1), U2.2 (A0), U2.7 (GND)
- net AS5600_SCL, INA226_SCL: now also U1.46 (PB9), R5.1; no longer U1.45 (PB8)
- net AS5600_SDA, INA226_SDA: now also U1.45 (PB8), R6.1; no longer U1.46 (PB9)
- net CONN1_DELTA: now also J1.2 (Pin_2), R8.1
- net CONN1_DRDY: now also J1.3 (Pin_3)
- net CONN1_GND: now also J1.1 (Pin_1)
- net CONN1_MISO: now also J1.4 (Pin_4)
- net CONN1_MOSI: now also J1.5 (Pin_5)
- net CONN1_NSS: now also J1.7 (Pin_7), R7.1
- net CONN1_SCLK: now also J1.6 (Pin_6)
- net USB_OTG_DM: now reaches U1.32 (PA11)
- net USB_OTG_DP: now reaches U1.33 (PA12)
- net JTAG_SWDIO: now reaches U1.34 (PA13)
- net JTAG_SWCLK: now reaches U1.37 (PA14)
- net at U1.44 (BOOT0): now also R1.1
- net RCC_OSC_IN: now reaches U1.5 (PH0)
- net RCC_OSC_OUT: now reaches U1.6 (PH1)
- net at U1.7 (NRST): now also R2.1, SW1.1
- net at U3.4 (FB): now also R3.1, R4.2
- net GND: now reaches U3.5 (~{ON}/OFF)
- net GND: now also A1.7 (GND), C1.2, C2.2, C3.2, C4.2, C5.2, C6.2, C7.2, C8.2, R4.1, SW1.2
- net +3V3: now reaches IC1.1 (VDD)
- net +3V3: now also A1.13 (~{RST}), A1.14 (~{SLP}), U1.24 (VDD), U2.6 (VDD), U3.2 (OUT), C5.1, C6.1, C7.1, C8.1, R2.2, R3.2, R5.2, R6.2, R7.2, R8.2
- net CONN2_A1 renamed CONN2_MOT_A1
- net CONN2_MOT_A1: now also J3.3 (Pin_3)
- net CONN2_A2 renamed CONN2_MOT_A2
- net CONN2_MOT_A2: now also J3.4 (Pin_4)
- net CONN2_B1 renamed CONN2_MOT_B1
- net CONN2_MOT_B1: now also J3.5 (Pin_5)
- net CONN2_B2 renamed CONN2_MOT_B2
- net CONN2_MOT_B2: now also J3.6 (Pin_6)
- net CONN2_GND: no longer names the net of U2.10 (VIN+)
- net CONN2_GND: no longer A1.7 (GND)
- net CONN2_VDD renamed +12V
- net +12V: now also C1.1, C2.1, C3.1, C4.1; no longer U2.9 (VIN-)
- removed net LM2596_OUT: A1.13 (~{RST}), A1.14 (~{SLP}), IC1.2 (VDD), U1.24 (VDD), U2.6 (VDD), U3.2 (OUT)
- new net CONN2_POWER+: J3.1 (Pin_1)
- new net CONN2_POWER-: J3.2 (Pin_2)
Other:
- moved on the sheet: A1, U1

Commit message: changes
Parts:
- added C10, C9: 100nF, symbol Device:C_Small
- added C11: 1uF, symbol Device:C_Polarized_Small
- added J2: USB_OTG, symbol Connector:USB_OTG
- added J4: Screw_Terminal_01x05, symbol Connector:Screw_Terminal_01x05
- added R10, R11: 10Ohm, symbol Device:R_Small
- added R9: 1Ohm, symbol Device:R_Small
- added Y1: ASCO, Oscillator:Oscillator_SMD_Abracon_ASCO-4Pin_1.6x1.2mm, symbol Oscillator:ASCO
- C5: value 10uF -> 100nF
- J1: value Screw_Terminal_01x07 -> CONN1
- J3: value Screw_Terminal_01x06 -> CONN2
- SW1: value SW_Push -> RESET
Connections:
- net AS5600_SCL, INA226_SCL is gone; now on net I2C1_SCL: R5.1, U1.46 (PB9)
- net AS5600_SDA, INA226_SDA is gone; now on net I2C1_SDA: R6.1, U1.45 (PB8)
- net CONN1_GND is gone; now on net GND: J1.1 (Pin_1)
- net CONN2_POWER+ is gone; now on net +12V: J3.1 (Pin_1)
- net INA226_SCL is gone; now on net I2C1_SCL: U2.5 (SCL)
- net INA226_SDA is gone; now on net I2C1_SDA: U2.4 (SDA)
- net +12V: now also U2.8 (VBUS), R10.1, R9.1
- net +3V3: now also C10.1, C9.1, J2.1 (VBUS), J4.1 (Pin_1), Y1.4 (VDD)
- net CONN1_DELTA: now also R7.1, U1.14 (PA4); no longer J1.2 (Pin_2), R8.1, U1.12 (PA2)
- net GND: now also C10.2, C9.2, J2.5 (GND), J4.2 (Pin_2), Y1.2 (GND); no longer A1.7 (GND), C3.2, C4.2
- net RCC_OSC_IN: now also Y1.3 (OUT)
- net SWNRST: now reaches R2.1, SW1.1, U1.7 (NRST)
- net SWNRST: now also R1.2, J4.5 (Pin_5)
- net at U2.10 (VIN+): now also C11.1, R10.2
- net at U2.9 (VIN-): now also C11.2, R11.2
- net AS5600_SCL renamed I2C1_SCL
- net AS5600_SDA renamed I2C1_SDA
- net CONN1_DRDY renamed DRDY
- net CONN1_MISO renamed SPI1_MISO
- net CONN1_MOSI renamed SPI1_MOSI
- removed net CONN1_NSS: J1.7 (Pin_7), R7.1, U1.14 (PA4)
- net CONN1_SCLK renamed SPI1_SCLK
- net CONN2_MOT_A1 renamed MOT_A1
- net CONN2_MOT_A2 renamed MOT_A2
- net CONN2_MOT_B1 renamed MOT_B1
- net CONN2_MOT_B2 renamed MOT_B2
- net CONN2_POWER- renamed GNDPWR
- net GNDPWR: now also A1.7 (GND), C3.2, C4.2, R11.1, R9.2
- net JTAG_SWCLK renamed SWCLK
- net SWCLK: now also J4.4 (Pin_4)
- net JTAG_SWDIO renamed SWDIO
- net SWDIO: now also J4.3 (Pin_3)
- net USB_OTG_DM renamed USB_OTG_D-
- net USB_OTG_D-: now also J2.2 (D-)
- net USB_OTG_DP renamed USB_OTG_D+
- net USB_OTG_D+: now also J2.3 (D+)
- new net DELTA: J1.2 (Pin_2)
- new net SPI1_NSS: J1.7 (Pin_7), R8.1, U1.12 (PA2)
Other:
- moved on the sheet: A1, C1, C2, C3, C4, C5, C6, C7, C8, IC1, J1, J3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

Commit message: changes
Parts:
- removed J4: Screw_Terminal_01x05, symbol Connector:Screw_Terminal_01x05
- removed Y1: ASCO, Oscillator:Oscillator_SMD_Abracon_ASCO-4Pin_1.6x1.2mm, symbol Oscillator:ASCO
- added J5: ARM_SWD_TC2030, Connector:Tag-Connect_TC2030-IDC-FP_2x03_P1.27mm_Vertical, symbol Connector:Conn_ARM_SWD_TagConnect_TC2030
- added Y1: ACO-25MHz, Oscillator:Oscillator_DIP-14, symbol Oscillator:ACO-xxxMHz
- renumbered C10 to C1, C11 to C10, C8 to C11, C6 to C2, C1 to C3, C2 to C4, C3 to C6, C4 to C7, C7 to C8, J2 to J1, J1 to J2, R5 to R1, R6 to R3, R1 to R4, R8 to R5, R4 to R6, R3 to R7, R7 to R8, U3 to U2, U2 to U3
Connections:
- net CONN1_DELTA is gone; now on net DELTA: R8.1, U1.14 (PA4)
- net GNDPWR is gone; now on net GND: A1.7 (GND), C6.2, C7.2, J3.2 (Pin_2), R11.1, R9.2
- net I2C1_SDA is gone; now on net I2C1_SCL: IC1.6 (SDA), R3.1, U1.45 (PB8), U3.4 (SDA)
- net +3V3: now also J5.1 (VCC), Y1.14 (Vcc)
- net DRV8825_DIR: now also U1.19 (PB1); no longer U1.40 (PB4)
- net DRV8825_EN: now also U1.18 (PB0); no longer U1.41 (PB5)
- net DRV8825_M0: now also U1.41 (PB5); no longer U1.18 (PB0)
- net DRV8825_M1: now also U1.40 (PB4); no longer U1.19 (PB1)
- net DRV8825_M2: now also U1.39 (PB3); no longer U1.20 (PB2)
- net DRV8825_STEP: now also U1.20 (PB2); no longer U1.39 (PB3)
- net GND: now also J1.6 (Shield), J5.5 (GND), Y1.7 (GND)
- net RCC_OSC_IN: now also Y1.8 (OUT)
- net SWCLK: now also J5.4 (SWCLK)
- net SWDIO: now also J5.2 (SWDIO)
- net SWNRST: now also J5.3 (~{RESET})
- net RCC_OSC_OUT: no longer names the net of U1.6 (PH1)
- no-connect marks 0 -> 28
Other:
- moved on the sheet: A1, C1, C10, C11, C2, C3, C4, C5, C6, C7, C8, C9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
