File: kicad_atlas_joint.kicad_pcb (KiCad board)
At the start: 2 copper layers, 6 parts, among them J5 ARM_SWD_TC2030, U1 STM32F411CEUx, U2 LM2596S-3.3, U3 INA226, Y1 ACO-25MHz

Commit message: changes
Parts:
- removed Y1: ACO-25MHz, Oscillator:Oscillator_DIP-14
- added C1: 100nF, Capacitor_SMD:C_0201_0603Metric_Pad0.64x0.40mm_HandSolder, F.Cu at (172.9, 90.7)
- added C10: 1uF, Capacitor_SMD:C_0201_0603Metric_Pad0.64x0.40mm_HandSolder, F.Cu at (147.9, 101.1)
- added C11: 100nF, Capacitor_SMD:C_0201_0603Metric_Pad0.64x0.40mm_HandSolder, F.Cu at (148.1, 98.4)
- added C12: 10pF, Capacitor_SMD:C_0201_0603Metric_Pad0.64x0.40mm_HandSolder, F.Cu at (158.4, 84.5)
- added C13: 10pF, Capacitor_SMD:C_0201_0603Metric_Pad0.64x0.40mm_HandSolder, F.Cu at (158.5, 83.1)
- added C2: 100nF, Capacitor_SMD:C_0201_0603Metric_Pad0.64x0.40mm_HandSolder, F.Cu at (121.6, 107.6)
- added C3: 10uF, Capacitor_SMD:C_0201_0603Metric_Pad0.64x0.40mm_HandSolder, F.Cu at (111.0, 87.0)
- added C4: 100nF, Capacitor_SMD:C_0201_0603Metric_Pad0.64x0.40mm_HandSolder, F.Cu at (111.0, 89.0)
- added C5: 100nF, Capacitor_SMD:C_0201_0603Metric_Pad0.64x0.40mm_HandSolder, F.Cu at (166.9, 90.6)
- added C6: 10uF, Capacitor_SMD:C_0201_0603Metric_Pad0.64x0.40mm_HandSolder, F.Cu at (106.0, 118.4)
- added C7: 100nF, Capacitor_SMD:C_0201_0603Metric_Pad0.64x0.40mm_HandSolder, F.Cu at (108.0, 118.4)
- added C8: 100nF, Capacitor_SMD:C_0201_0603Metric_Pad0.64x0.40mm_HandSolder, F.Cu at (147.2, 92.4)
- added C9: 100nF, Capacitor_SMD:C_0201_0603Metric_Pad0.64x0.40mm_HandSolder, F.Cu at (161.0, 93.9)
- added IC1: AS5600-ASOT, as5600:SOIC127P600X175-8N, F.Cu at (152.5, 93.0)
- added J1: USB_C_Receptacle_USB2.0_16P, Connector_USB:USB_C_Receptacle_JAE_DX07S016JA1R1500, F.Cu at (164.0, 100.0)
- added J2: CONN1, Connector_JST:JST_SHL_SM07B-SHLS-TF_1x07-1MP_P1.00mm_Horizontal, F.Cu at (176.5, 99.0)
- added J3: CONN2, TerminalBlock:TerminalBlock_Xinya_XY308-2.54-6P_1x06_P2.54mm_Horizontal, F.Cu at (115.8, 84.0)
- added R1: 4.7kOhm, Resistor_SMD:R_0201_0603Metric, F.Cu at (163.0, 79.2)
- added R10: 10Ohm, Resistor_SMD:R_0201_0603Metric, F.Cu at (146.4, 102.4)
- added R11: 10Ohm, Resistor_SMD:R_0201_0603Metric, F.Cu at (146.3, 99.7)
- added R12: 5kOhm, Resistor_SMD:R_0201_0603Metric, F.Cu at (163.0, 94.0)
- added R13: 5kOhm, Resistor_SMD:R_0201_0603Metric, F.Cu at (165.0, 94.0)
- added R2: 10kOhm, Resistor_SMD:R_0201_0603Metric, F.Cu at (158.4, 85.9)
- added R3: 4.7kOhm, Resistor_SMD:R_0201_0603Metric, F.Cu at (161.5, 79.2)
- added R4: 10kOhm, Resistor_SMD:R_0201_0603Metric, F.Cu at (164.5, 79.2)
- added R5: 10kOhm, Resistor_SMD:R_0201_0603Metric, F.Cu at (158.4, 87.4)
- added R6: 1.7kOhm, Resistor_SMD:R_0201_0603Metric, F.Cu at (108.0, 116.4)
- added R7: 1kOhm, Resistor_SMD:R_0201_0603Metric, F.Cu at (108.0, 113.5)
- added R8: 10kOhm, Resistor_SMD:R_0201_0603Metric, F.Cu at (162.0, 90.4)
- added R9: 1Ohm, Resistor_SMD:R_0201_0603Metric, F.Cu at (144.9, 101.1)
- added SW1: RESET, Resistor_SMD:R_0201_0603Metric, F.Cu at (158.3, 81.0)
- added Y2: Crystal, Crystal:Crystal_AT310_D3.0mm_L10.0mm_Horizontal, B.Cu at (156.0, 85.3)
- moved U2 54.8 mm to (119.4, 115.0)
- moved U1 34.2 mm to (164.2, 84.8)
- moved A1 22.9 mm to (128.9, 91.7), turned to -90 degrees
- moved U3 19.5 mm to (152.7, 99.5), turned to 180 degrees
- moved J5 7.97 mm to (174.9, 84.5)
Connections:
- U1 pad 45: /I2C1_SCL -> /I2C1_SDA
- U1 pad 6: unconnected-(U1-PH1-Pad6) -> /RCC_OSC_OUT
- U3 pad 4: /I2C1_SCL -> /I2C1_SDA

Commit message: changes
Parts:
- moved J5 36.9 mm to (138.0, 84.1), turned to 90 degrees
- moved R4 35.2 mm to (132.8, 94.5), turned to 180 degrees
- moved R1 34.6 mm to (132.8, 96.0), turned to 180 degrees
- moved R3 34.1 mm to (132.7, 97.5), turned to 180 degrees
- moved SW1 30.9 mm to (134.6, 100.7), turned to 90 degrees
- moved J2 29.7 mm to (151.5, 83.0), turned to 0 degrees
- moved C1 29.0 mm to (144.3, 86.1), turned to 90 degrees
- moved C13 28.0 mm to (136.6, 100.5), turned to -90 degrees
- moved U1 27.8 mm to (138.3, 94.8), turned to 90 degrees
- moved C12 26.0 mm to (138.1, 100.6), turned to -90 degrees
- moved Y2 24.6 mm to (138.9, 103.0), turned to 180 degrees
- moved R2 24.0 mm to (139.4, 100.6), turned to -90 degrees
- moved C5 22.8 mm to (144.1, 92.1), turned to 0 degrees
- moved R5 21.9 mm to (140.9, 100.6), turned to -90 degrees
- moved C8 19.4 mm to (145.9, 111.8), turned to -90 degrees
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